Commit message: Imported upstream version '0.1.0' of 'upstream'

File: warthog_description/urdf/accessories/novatel_smart6.urdf.xacro (robot description, xacro)
@@ -1,4 +1,4 @@
 <?xml version="1.0"?>
-<robot xmlns:xacro="http://ros.org/wiki/xacro">
+<robot xmlns:xacro="http://www.ros.org/wiki/xacro">
   <xacro:macro name="novatel_smart6" params="prefix">
   <link name="${prefix}_link">

File: warthog_description/urdf/accessories/warthog_bulkhead.urdf.xacro (robot description, xacro)
@@ -1,4 +1,4 @@
 <?xml version="1.0"?>
-<robot xmlns:xacro="http://ros.org/wiki/xacro">
+<robot xmlns:xacro="http://www.ros.org/wiki/xacro">
   <xacro:macro name="warthog_bulkhead">
     <link name="bulkhead_link">

File: warthog_description/urdf/warthog.urdf.xacro (robot description, xacro)
@@ -76,8 +76,8 @@
       <type>transmission_interface/SimpleTransmission</type>
       <joint name="${prefix}_${side}_wheel_joint">
-        <hardwareInterface>VelocityJointInterface</hardwareInterface>
+        <hardwareInterface>hardware_interface/VelocityJointInterface</hardwareInterface>
       </joint>
       <actuator name="${prefix}_${side}_actuator">
-        <hardwareInterface>VelocityJointInterface</hardwareInterface>
+        <hardwareInterface>hardware_interface/VelocityJointInterface</hardwareInterface>
         <mechanicalReduction>1</mechanicalReduction>
       </actuator>
@@ -124,8 +124,8 @@
       <type>transmission_interface/SimpleTransmission</type>
       <joint name="${prefix}_${side}_wheel_joint">
-        <hardwareInterface>VelocityJointInterface</hardwareInterface>
+        <hardwareInterface>hardware_interface/VelocityJointInterface</hardwareInterface>
       </joint>
       <actuator name="${prefix}_${side}_actuator">
-        <hardwareInterface>VelocityJointInterface</hardwareInterface>
+        <hardwareInterface>hardware_interface/VelocityJointInterface</hardwareInterface>
         <mechanicalReduction>1</mechanicalReduction>
       </actuator>
@@ -204,5 +204,5 @@
     </link>
     <joint name="${prefix}_diff_unit_joint" type="revolute">
-      <limit upper="0.15" lower="-0.15" effort="100000" velocity="1"/>
+      <limit upper="0.4" lower="-0.4" effort="100" velocity="1"/>
       <parent link="chassis_link"/>
       <child link="${prefix}_diff_unit_link"/>
