Commit message: Imported upstream version '0.0.2' of 'upstream'

File: warthog_description/urdf/accessories.urdf.xacro (robot description, xacro)
@@ -9,3 +9,37 @@
     warthog_base/launch/base.launch
   -->
+  <!-- If enabled, generate a Novatel Smart6 payload. -->
+  <xacro:include filename="accessories/novatel_smart6.urdf.xacro" />
+  <xacro:if value="$(optenv WARTHOG_NAVSAT_SMART6 0)">
+    <novatel_smart6 prefix="$(optenv WARTHOG_NAVSAT_SMART6_MOUNT navsat)"/>
+    <joint name="$(optenv WARTHOG_NAVSAT_SMART6_MOUNT navsat)_joint" type="fixed">
+    <origin xyz="$(optenv WARTHOG_NAVSAT_SMART6_OFFSET 0 0 0)"
+            rpy="$(optenv WARTHOG_NAVSAT_SMART6_RPY 0 0 0)" />
+      <parent link="top_chassis_link" />
+      <child link="$(optenv WARTHOG_NAVSAT_SMART6_MOUNT navsat)_link" />
+    </joint>
+  </xacro:if>
+  <xacro:include filename="accessories/warthog_bulkhead.urdf.xacro" />
+  <xacro:if value="$(optenv WARTHOG_BULKHEAD 0)">
+    <warthog_bulkhead/>
+    <joint name="bulkhead_link_joint" type="fixed">
+      <origin xyz="0.00705 0 0.24184" rpy="0 0 0" />
+      <parent link="top_chassis_link"/>
+      <child link="bulkhead_link" />
+    </joint>
+    <joint name="bulkhead_front_mount_link_joint" type="fixed">
+      <origin xyz="0.33987 0 0.0" rpy="0 0 0" />
+      <parent link="bulkhead_link"/>
+      <child link="bulkhead_front_mount_link" />
+    </joint>
+        <xacro:include filename="accessories/warthog_arm_mount.urdf.xacro" />
+        <xacro:if value="$(optenv WARTHOG_ARM_MOUNT 0)">
+          <warthog_arm_mount/>
+          <joint name="arm_mount_link_joint" type="fixed">
+            <origin xyz="0 0 0.02" rpy="0 0 0" />
+            <parent link="bulkhead_front_mount_link"/>
+            <child link="arm_mount_link" />
+          </joint>
+        </xacro:if>
+  </xacro:if>
 </robot>

File: warthog_description/urdf/accessories/novatel_smart6.urdf.xacro (robot description, xacro)
@@ -1,6 +1,6 @@
 <?xml version="1.0"?>
 <robot xmlns:xacro="http://ros.org/wiki/xacro">
-  <xacro:macro name="novatel_smart6">
-  <link name="navsat_link">
+  <xacro:macro name="novatel_smart6" params="prefix">
+  <link name="${prefix}_link">
     <visual>
       <origin xyz="0 0 0" rpy="0 0 0" />

File: warthog_description/urdf/warthog.urdf.xacro (robot description, xacro)
@@ -4,6 +4,8 @@
   <material name="dark_grey"><color rgba="0.2 0.2 0.2 1.0" /></material>
   <material name="light_grey"><color rgba="0.4 0.4 0.4 1.0" /></material>
-  <material name="yellow"><color rgba="0.8 0.8 0.0 1.0" /></material>
+  <material name="yellow"><color rgba="0.95 0.816 0.082 1.0" /></material>
   <material name="black"><color rgba="0.15 0.15 0.15 1.0" /></material>
+  <material name="white"><color rgba="0.9 0.9 0.9 1.0" /></material>
+  <material name="red"><color rgba="0.9 0.0 0.0 1.0" /></material>
   <xacro:macro name="wheel" params="prefix side fwd left">
     <link name="${prefix}_wheel">
@@ -14,5 +16,5 @@
       </inertial>
       <visual>
-        <origin xyz="0 0 0" rpy="0 0 ${PI/2}"/>
+        <origin xyz="0 0 0" rpy="0 0 ${side*PI/2}"/>
         <geometry>
           <mesh filename="package://warthog_description/meshes/wheel.stl" />
@@ -21,5 +23,5 @@
       </visual>
       <collision>
-        <origin xyz="0 0 0" rpy="${PI/2} 0 0"/>
+        <origin xyz="0 0 0" rpy="${side*PI/2} 0 0"/>
         <geometry>
           <cylinder radius="${wheel_radius}" length="${wheel_width}"/>
@@ -71,14 +73,35 @@
       </inertial>
       <visual>
-        <origin xyz="0 ${side*-1*0.05} 0.197" rpy="${PI/2} 0 ${PI/2-side*PI/2}"/>
+        <origin xyz="0 0 0" rpy="0 0 ${side*PI/2}"/>
         <geometry>
           <mesh filename="package://warthog_description/meshes/rocker.stl" />
         </geometry>
-        <material name="yellow" />
+        <material name="black"><color rgba="0.15 0.15 0.15 1.0" /></material>
+      </visual>
+      <visual>
+        <origin xyz="0 0 0" rpy="0 0 ${side*PI/2}"/>
+        <geometry>
+          <mesh filename="package://warthog_description/meshes/fenders.stl" />
+        </geometry>
+        <material name="yellow"><color rgba="0.95 0.816 0.082 1.0" /></material>
+      </visual>
+      <visual>
+        <origin xyz="0 ${side*-0.0244} 0" rpy="0 0 0"/>
+        <geometry>
+          <mesh filename="package://warthog_description/meshes/light.stl" />
+        </geometry>
+        <material name="white"><color rgba="0.9 0.9 0.9 1.0" /></material>
+      </visual>
+      <visual>
+        <origin xyz="0 ${side*-0.0244} 0" rpy="0 0 ${side*PI}"/>
+        <geometry>
+          <mesh filename="package://warthog_description/meshes/light.stl" />
+        </geometry>
+        <material name="red"><color rgba="0.9 0.0 0.0 1.0" /></material>
       </visual>
       <collision>
-        <origin xyz="0 0 0.197" rpy="0 0 0"/>
-        <geometry>
-          <box size="${diff_unit_length} ${diff_unit_width} ${diff_unit_height}"/>
+        <origin xyz="0 0 0" rpy="0 0 ${side*PI/2}"/>
+        <geometry>
+          <mesh filename="package://warthog_description/meshes/fenders.stl" />
         </geometry>
       </collision>
@@ -86,5 +109,5 @@
     <joint name="${prefix}_diff_unit_jnt" type="revolute">
       <limit upper="0.15" lower="-0.15" effort="100000" velocity="1"/>
-      <parent link="base_link"/>
+      <parent link="chassis_link"/>
       <child link="${prefix}_diff_unit_link"/>
       <origin xyz="${diff_unit_offset_x} ${diff_unit_offset_y*side} ${diff_unit_offset_z}" rpy="0 0 0" />
@@ -94,10 +117,16 @@
     <gazebo reference="${prefix}_diff_unit_link">
       <selfCollide>false</selfCollide>
-      <material>Gazebo/Orange</material>
+      <material>Gazebo/Yellow</material>
     </gazebo>
   </xacro:macro>
   <xacro:diff_unit prefix="left" side="1" left="true"/>
   <xacro:diff_unit prefix="right" side="-1" left="false"/>
-  <link name="base_link">
+  <link name="base_link"></link>
+  <joint name="base_link_joint" type="fixed">
+    <origin xyz="0 0 0.025" rpy="0 0 0" />
+    <parent link="base_link"/>
+    <child link="chassis_link" />
+  </joint>
+  <link name="chassis_link">
     <inertial>
       <origin xyz="0 0 0" rpy="0 0 0"/>
@@ -111,21 +140,30 @@
         <mesh filename="package://warthog_description/meshes/chassis.stl" />
       </geometry>
-      <material name="black" />
+      <material name="black"><color rgba="0.15 0.15 0.15 1.0" /></material>
+    </visual>
+    <visual>
+      <origin xyz="0 0 0" rpy="0 0 0"/>
+      <geometry>
+        <mesh filename="package://warthog_description/meshes/e-stop.stl" />
+      </geometry>
+      <material name="red"><color rgba="0.9 0.0 0.0 1.0" /></material>
     </visual>
     <collision>
       <origin xyz="0 0 0" rpy="0 0 0"/>
       <geometry>
-        <box size="${chassis_length} ${chassis_width} ${chassis_height}"/>
+        <mesh filename="package://warthog_description/meshes/chassis-collision.stl" />
       </geometry>
     </collision>
   </link>
-  <gazebo reference="base_link">
-    <selfCollide>false</selfCollide>
-    <material>Gazebo/Orange</material>
-  </gazebo>
+  <link name="top_chassis_link"></link>
+  <joint name="top_link_joint" type="fixed">
+    <origin xyz="0 0 0.27218" rpy="0 0 0" />
+    <parent link="chassis_link"/>
+    <child link="top_chassis_link" />
+  </joint>
   <!-- This link is purely to complete the visual look -->
   <link name="diff_link">
     <visual>
-      <origin xyz="0 0 0" rpy="0 0 ${PI/2}"/>
+      <origin xyz="0 0 0" rpy="0 0 0"/>
       <geometry>
         <mesh filename="package://warthog_description/meshes/diff-link.stl" />
@@ -134,5 +172,5 @@
     </visual>
     <visual>
-      <origin xyz="0.285 0.3845 0.008" rpy="0 ${PI/2} 0"/>
+      <origin xyz="0 0 0" rpy="0 0 0"/>
       <geometry>
         <mesh filename="package://warthog_description/meshes/susp-link.stl" />
@@ -141,5 +179,5 @@
     </visual>
     <visual>
-      <origin xyz="0.285 0.3845 0.008" rpy="0 ${PI/2} 0"/>
+      <origin xyz="0 0 0" rpy="0 0 0"/>
       <geometry>
         <mesh filename="package://warthog_description/meshes/susp-link.stl" />
@@ -148,12 +186,15 @@
     </visual>
   </link>
-  <joint name="$diff_link_jnt" type="fixed">
-    <parent link="base_link"/>
+  <joint name="diff_link_jnt" type="fixed">
+    <parent link="chassis_link"/>
     <child link="diff_link"/>
-    <origin xyz="-0.65 0 0.07" rpy="0 0 0" />
-  </joint>
-  <gazebo reference="diff_link">
-    <material>Gazebo/Grey</material>
-  </gazebo>
+    <origin xyz="-0.5826 0 0.24979" rpy="0 0 0" />
+  </joint>
+  <link name="imu_link" />
+  <joint name="imu_link_joint" type="fixed">
+    <origin xyz="$(optenv WARTHOG_IMU_XYZ 0 0 0)" rpy="$(optenv WARTHOG_IMU_RPY 0 0 0)" />
+    <parent link="chassis_link"/>
+    <child link="imu_link" />
+  </joint>
   <!-- Bring in simulation data for Gazebo. -->
   <xacro:include filename="$(find warthog_description)/urdf/warthog.gazebo" />
@@ -163,4 +204,4 @@
   <xacro:include filename="$(find warthog_description)/urdf/accessories.urdf.xacro" />
   <!-- Optional custom includes. -->
-  <xacro:include filename="$(find warthog_description)/urdf/$(optenv WARTHOG_URDF_EXTRAS empty.urdf)" />
+  <xacro:include filename="$(optenv WARTHOG_URDF_EXTRAS empty.urdf)" />
 </robot>

File: warthog_description/urdf/warthog_params.xacro (robot description, xacro)
@@ -5,14 +5,14 @@
   <xacro:property name="wheel_width" value="0.25" />
   <xacro:property name="wheel_mass" value="15" />
-  <xacro:property name="axle_x_offset" value="0.46" />
-  <xacro:property name="axle_y_offset" value="0.01" />
-  <xacro:property name="axle_z_offset" value="-0.005" />
+  <xacro:property name="axle_x_offset" value="0.457367" />
+  <xacro:property name="axle_y_offset" value="0.0" />
+  <xacro:property name="axle_z_offset" value="-0.012977" />
   <xacro:property name="diff_unit_length" value="1.34" />
   <xacro:property name="diff_unit_width" value="0.28" />
   <xacro:property name="diff_unit_height" value="0.63"/>
   <xacro:property name="diff_unit_mass" value="50" />
-  <xacro:property name="diff_unit_offset_x" value="0.04" />
-  <xacro:property name="diff_unit_offset_y" value="0.55" />
-  <xacro:property name="diff_unit_offset_z" value="-0.105" />
+  <xacro:property name="diff_unit_offset_x" value="0.00" />
+  <xacro:property name="diff_unit_offset_y" value="0.56821" />
+  <xacro:property name="diff_unit_offset_z" value="0.0" />
   <xacro:property name="chassis_length" value="1.35" />
   <xacro:property name="chassis_width" value="0.70" />

Commit message: Imported upstream version '0.0.3' of 'upstream'

File: warthog_description/urdf/accessories.urdf.xacro (robot description, xacro)
@@ -33,13 +33,13 @@
       <child link="bulkhead_front_mount_link" />
     </joint>
-        <xacro:include filename="accessories/warthog_arm_mount.urdf.xacro" />
-        <xacro:if value="$(optenv WARTHOG_ARM_MOUNT 0)">
-          <warthog_arm_mount/>
-          <joint name="arm_mount_link_joint" type="fixed">
-            <origin xyz="0 0 0.02" rpy="0 0 0" />
-            <parent link="bulkhead_front_mount_link"/>
-            <child link="arm_mount_link" />
-          </joint>
-        </xacro:if>
+    <xacro:include filename="accessories/warthog_arm_mount.urdf.xacro" />
+    <xacro:if value="$(optenv WARTHOG_ARM_MOUNT 0)">
+    <warthog_arm_mount/>
+    <joint name="arm_mount_link_joint" type="fixed">
+      <origin xyz="0 0 0.02" rpy="0 0 0" />
+      <parent link="bulkhead_front_mount_link"/>
+      <child link="arm_mount_link" />
+    </joint>
+    </xacro:if>
   </xacro:if>
 </robot>

File: warthog_description/urdf/warthog.urdf.xacro (robot description, xacro)
@@ -1,5 +1,34 @@
 <?xml version='1.0'?>
 <robot name="warthog" xmlns:xacro="http://www.ros.org/wiki/xacro">
-  <xacro:include filename="$(find warthog_description)/urdf/warthog_params.xacro" />
+  <xacro:property name="PI" value="3.1415926535897931"/>
+  <xacro:property name="wheel_radius" value="0.3" />
+  <xacro:property name="wheel_width" value="0.25" />
+  <xacro:property name="wheel_mass" value="15" />
+  <xacro:property name="wheel_to_track_ratio" value="0.5962" />
+  <xacro:property name="axle_x_offset" value="0.457367" />
+  <xacro:property name="axle_y_offset" value="0.0" />
+  <xacro:property name="axle_z_offset" value="-0.012977" />
+  <xacro:property name="diff_unit_length" value="1.34" />
+  <xacro:property name="diff_unit_width" value="0.28" />
+  <xacro:property name="diff_unit_height" value="0.63"/>
+  <xacro:property name="diff_unit_mass" value="50" />
+  <xacro:property name="diff_unit_offset_x" value="0.00" />
+  <xacro:property name="diff_unit_offset_y" value="0.56821" />
+  <xacro:property name="diff_unit_offset_z" value="0.0" />
+  <xacro:property name="chassis_length" value="1.35" />
+  <xacro:property name="chassis_width" value="0.70" />
+  <xacro:property name="chassis_height" value="0.30" />
+  <xacro:property name="chassis_mass" value="100" />
+  <xacro:property name="dummy_inertia" value="1e-09"/>
+  <xacro:macro name="wheel_inertia" params="m r h">
+    <inertia ixx="${m*(3*r*r+h*h)/12}" ixy="0" ixz="0"
+             iyy="${m*r*r/2}" iyz="0"
+             izz="${m*(3*r*r+h*h)/12}" />
+  </xacro:macro>
+  <xacro:macro name="box_inertia" params="m x y z">
+    <inertia ixx="${m*(y*y+z*z)/12}" ixy="0" ixz="0"
+             iyy="${m*(x*x+z*z)/12}" iyz="0"
+             izz="${m*(x*x+z*z)/12}" />
+  </xacro:macro>
   <material name="dark_grey"><color rgba="0.2 0.2 0.2 1.0" /></material>
   <material name="light_grey"><color rgba="0.4 0.4 0.4 1.0" /></material>
@@ -8,6 +37,6 @@
   <material name="white"><color rgba="0.9 0.9 0.9 1.0" /></material>
   <material name="red"><color rgba="0.9 0.0 0.0 1.0" /></material>
-  <xacro:macro name="wheel" params="prefix side fwd left">
-    <link name="${prefix}_wheel">
+  <xacro:macro name="wheel" params="prefix side *joint_pose">
+    <link name="${prefix}_${side}_wheel_link">
       <inertial>
         <origin xyz="0 0 0" rpy="0 0 0" />
@@ -16,5 +45,5 @@
       </inertial>
       <visual>
-        <origin xyz="0 0 0" rpy="0 0 ${side*PI/2}"/>
+        <origin xyz="0 0 0" rpy="0 0 ${PI/2}"/>
         <geometry>
           <mesh filename="package://warthog_description/meshes/wheel.stl" />
@@ -23,5 +52,5 @@
       </visual>
       <collision>
-        <origin xyz="0 0 0" rpy="${side*PI/2} 0 0"/>
+        <origin xyz="0 0 0" rpy="${PI/2} 0 0"/>
         <geometry>
           <cylinder radius="${wheel_radius}" length="${wheel_width}"/>
@@ -29,16 +58,11 @@
       </collision>
     </link>
-    <joint name="${prefix}_wheel_jnt" type="continuous">
-      <xacro:if value="${left}">
-        <parent link="left_diff_unit_link"/>
-      </xacro:if>
-      <xacro:unless value="${left}">
-        <parent link="right_diff_unit_link"/>
-      </xacro:unless>
-      <child link="${prefix}_wheel"/>
-      <origin xyz="${axle_x_offset*fwd} ${axle_y_offset*side} ${axle_z_offset}" rpy="0 0 0" />
+    <joint name="${prefix}_${side}_wheel_joint" type="continuous">
+      <parent link="${side}_diff_unit_link"/>
+      <child link="${prefix}_${side}_wheel_link"/>
+      <xacro:insert_block name="joint_pose" />
       <axis xyz="0 1 0"/>
     </joint>
-    <gazebo reference="${prefix}_wheel">
+    <gazebo reference="${prefix}_${side}_wheel_link">
       <selfCollide>false</selfCollide>
       <mu1>0.9</mu1>
@@ -49,10 +73,10 @@
       <material>Gazebo/Grey</material>
     </gazebo>
-    <transmission name="${prefix}_wheel_trans">
+    <transmission name="${prefix}_${side}_wheel_trans">
       <type>transmission_interface/SimpleTransmission</type>
-      <joint name="${prefix}_wheel_jnt">
+      <joint name="${prefix}_${side}_wheel_joint">
         <hardwareInterface>VelocityJointInterface</hardwareInterface>
       </joint>
-      <actuator name="${prefix}_actuator">
+      <actuator name="${prefix}_${side}_actuator">
         <hardwareInterface>VelocityJointInterface</hardwareInterface>
         <mechanicalReduction>1</mechanicalReduction>
@@ -60,8 +84,80 @@
     </transmission>
   </xacro:macro>
-  <xacro:wheel prefix="fl" side="1" fwd="1" left="true"/>
-  <xacro:wheel prefix="fr" side="-1" fwd="1" left="false"/>
-  <xacro:wheel prefix="bl" side="1" fwd="-1" left="true"/>
-  <xacro:wheel prefix="br" side="-1" fwd="-1" left="false"/>
+  <xacro:macro name="track" params="prefix side *joint_pose">
+    <link name="${prefix}_${side}_track_link">
+      <visual>
+        <origin xyz="0 0 0" rpy="0 0 0"/>
+        <geometry>
+          <mesh filename="package://warthog_description/meshes/tracks.dae" />
+        </geometry>
+        <material name="dark_grey" />
+      </visual>
+      <collision>
+        <origin xyz="0 0 0" rpy="0 0 0"/>
+        <geometry>
+          <mesh filename="package://warthog_description/meshes/tracks_collision.stl" />
+        </geometry>
+      </collision>
+    </link>
+    <joint name="${prefix}_${side}_track_joint" type="fixed">
+      <parent link="${side}_diff_unit_link"/>
+      <child link="${prefix}_${side}_track_link"/>
+      <xacro:insert_block name="joint_pose" />
+      <axis xyz="0 1 0"/>
+    </joint>
+    <!-- This adds wheels that rotate instead of tracks. -->
+    <link name="${prefix}_${side}_wheel_link">
+      <collision>
+        <origin xyz="0 0 0" rpy="${PI/2} 0 0"/>
+        <geometry>
+          <cylinder radius="${wheel_radius*wheel_to_track_ratio}" length="${wheel_width}"/>
+        </geometry>
+      </collision>
+    </link>
+    <joint name="${prefix}_${side}_wheel_joint" type="continuous">
+      <parent link="${side}_diff_unit_link"/>
+      <child link="${prefix}_${side}_wheel_link"/>
+      <xacro:insert_block name="joint_pose" />
+      <axis xyz="0 1 0"/>
+    </joint>
+    <transmission name="${prefix}_${side}_wheel_trans">
+      <type>transmission_interface/SimpleTransmission</type>
+      <joint name="${prefix}_${side}_wheel_joint">
+        <hardwareInterface>VelocityJointInterface</hardwareInterface>
+      </joint>
+      <actuator name="${prefix}_${side}_actuator">
+        <hardwareInterface>VelocityJointInterface</hardwareInterface>
+        <mechanicalReduction>1</mechanicalReduction>
+      </actuator>
+    </transmission>
+  </xacro:macro>
+  <xacro:unless value="$(optenv WARTHOG_TRACKS 0)">
+    <xacro:wheel prefix="front" side="left">
+      <origin xyz="${axle_x_offset*1} ${axle_y_offset*1} ${axle_z_offset}" rpy="0 0 0" />
+    </xacro:wheel>
+    <xacro:wheel prefix="front" side="right">
+      <origin xyz="${axle_x_offset*1} ${axle_y_offset*-1} ${axle_z_offset}" rpy="0 0 0" />
+    </xacro:wheel>
+    <xacro:wheel prefix="rear" side="left">
+      <origin xyz="${axle_x_offset*-1} ${axle_y_offset*1} ${axle_z_offset}" rpy="0 0 0" />
+    </xacro:wheel>
+    <xacro:wheel prefix="rear" side="right">
+      <origin xyz="${axle_x_offset*-1} ${axle_y_offset*-1} ${axle_z_offset}" rpy="0 0 0" />
+    </xacro:wheel>
+  </xacro:unless>
+  <xacro:if value="$(optenv WARTHOG_TRACKS 0)">
+    <xacro:track prefix="front" side="left">
+      <origin xyz="${axle_x_offset*1} ${axle_y_offset*1} ${axle_z_offset}" rpy="0 0 0" />
+    </xacro:track>
+    <xacro:track prefix="front" side="right">
+      <origin xyz="${axle_x_offset*1} ${axle_y_offset*-1} ${axle_z_offset}" rpy="0 0 0" />
+    </xacro:track>
+    <xacro:track prefix="rear" side="left">
+      <origin xyz="${axle_x_offset*-1} ${axle_y_offset*1} ${axle_z_offset}" rpy="0 0 ${PI}" />
+    </xacro:track>
+    <xacro:track prefix="rear" side="right">
+      <origin xyz="${axle_x_offset*-1} ${axle_y_offset*-1} ${axle_z_offset}" rpy="0 0 ${PI}" />
+    </xacro:track>
+  </xacro:if>
   <xacro:macro name="diff_unit" params="prefix side left">
     <link name="${prefix}_diff_unit_link">
@@ -107,5 +203,5 @@
       </collision>
     </link>
-    <joint name="${prefix}_diff_unit_jnt" type="revolute">
+    <joint name="${prefix}_diff_unit_joint" type="revolute">
       <limit upper="0.15" lower="-0.15" effort="100000" velocity="1"/>
       <parent link="chassis_link"/>
@@ -186,5 +282,5 @@
     </visual>
   </link>
-  <joint name="diff_link_jnt" type="fixed">
+  <joint name="diff_link_joint" type="fixed">
     <parent link="chassis_link"/>
     <child link="diff_link"/>

Commit message: Imported upstream version '0.1.4' of 'upstream'

File: warthog_description/urdf/accessories.urdf.xacro (robot description, xacro)
@@ -18,4 +18,13 @@
       <parent link="top_chassis_link" />
       <child link="$(optenv WARTHOG_NAVSAT_SMART6_MOUNT navsat)_link" />
+    </joint>
+  </xacro:if>
+  <xacro:include filename="accessories/warthog_generator.urdf.xacro" />
+  <xacro:if value="$(optenv WARTHOG_GENERATOR 0)">
+    <xacro:warthog_generator/>
+    <joint name="generator_link_joint" type="fixed">
+      <origin xyz="-0.42506 0 0.0017" rpy="0 0 0" />
+      <parent link="top_chassis_link"/>
+      <child link="generator_link" />
     </joint>
   </xacro:if>

File: warthog_description/urdf/warthog.urdf.xacro (robot description, xacro)
@@ -21,4 +21,25 @@
   <xacro:property name="chassis_mass" value="100" />
   <xacro:property name="dummy_inertia" value="1e-09"/>
+  <!--
+    Optional paint colors.
+    Available colors:
+      - yellow (default)
+      - orange
+      - olive
+      - sand
+  -->
+  <xacro:property name="warthog_color" value="$(optenv WARTHOG_COLOR yellow)" />
+  <xacro:if value="${warthog_color == 'yellow'}">
+    <xacro:property name="warthog_color_rgba" value="0.95 0.816 0.082 1.0" />
+  </xacro:if>
+  <xacro:if value="${warthog_color == 'orange'}">
+    <xacro:property name="warthog_color_rgba" value="1.0 0.48 0.0 1.0" />
+  </xacro:if>
+  <xacro:if value="${warthog_color == 'olive'}">
+    <xacro:property name="warthog_color_rgba" value="0.333 0.419 0.184 1.0" />
+  </xacro:if>
+  <xacro:if value="${warthog_color == 'sand'}">
+    <xacro:property name="warthog_color_rgba" value="0.86 0.75 0.54 1.0" />
+  </xacro:if>
   <xacro:macro name="wheel_inertia" params="m r h">
     <inertia ixx="${m*(3*r*r+h*h)/12}" ixy="0" ixz="0"
@@ -180,5 +201,7 @@
           <mesh filename="package://warthog_description/meshes/fenders.stl" />
         </geometry>
-        <material name="yellow"><color rgba="0.95 0.816 0.082 1.0" /></material>
+        <material name="${warthog_color}">
+          <color rgba="${warthog_color_rgba}" />
+        </material>
       </visual>
       <visual>
@@ -301,3 +324,5 @@
   <!-- Optional custom includes. -->
   <xacro:include filename="$(optenv WARTHOG_URDF_EXTRAS empty.urdf)" />
+  <!-- Optional for Clearpath internal softwares -->
+  <xacro:include filename="$(optenv CPR_URDF_EXTRAS empty.urdf)" />
 </robot>
